File: MIDI_IN/MIDI_IN.kicad_pcb (KiCad board)
At the start: 2 copper layers, 20.3 x 62 mm, 13 parts, among them J1 DIN-5 Midi Jack, J2 TO MCU, J3 MIDI THRU, U1 6N137

Commit message: Updated license to CERN-OHL-P v2 license
Signed-off-by: CTXz <ctx.xda@gmail.com>
Parts:
- moved C1 52.7 mm to (74.8, 50.5)
- moved D1 52.7 mm to (59.6, 61.4)
- moved J2 52.7 mm to (60.8, 45.4)
- moved J3 52.7 mm to (69.2, 40.4)
- moved R2 52.7 mm to (74.8, 53.5)
- moved REF** 52.7 mm to (72.9, 33.7)
- moved U1 52.7 mm to (63.6, 58.4)
- moved J1 52.7 mm to (67.2, 82.0)
- moved R1 52.7 mm to (74.8, 69.1)
- moved REF** 52.7 mm to (61.4, 33.7)
- moved REF** 52.7 mm to (67.2, 65.3)
- moved REF** 52.7 mm to (67.2, 64.5)
- moved C2 52.7 mm to (59.5, 58.3)
Other:
- board text added: "Patrick Pedersen Licensed under CERN-OHL-P v2 Made in the TU-DO Makerspace"
- board text removed: "Patrick Pedersen TAPR Open Hardware License v1.0 Made in the TU-DO Makerspace"
