File: MIDI_OUT/MIDI_OUT.kicad_pcb (KiCad board)
At the start: 2 copper layers, 20.3 x 50.9 mm, 15 parts, among them J1 Conn_01x03_Male, J2 DIN-5_180degree, Q1 BS170, Q2 BS170, SW1 SW_Push_DPDT

Commit message: Updated license to CERN-OHL-P v2 license
Signed-off-by: CTXz <ctx.xda@gmail.com>
Other:
- board text added: "Patrick Pedersen Licensed under CERN-OHL-P v2"
- board text removed: "Patrick Pedersen TAPR Open Hardware License v1.0"
Changed lines of the file:
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@@
   (title_block
     (title "MIDI Output Breakout Board")
-    (date "2022-09-11")
-    (rev "2.0")
+    (date "2022-11-14")
+    (rev "2.1")
     (company "TU-DO Makerspace")
-    (comment 1 "License: TAPR Open Hardware License v1.0")
+    (comment 1 "License: CERN-OHL-P v2")
     (comment 2 "ctx.xda@gmail.com")
     (comment 3 "Author: Patrick Pedersen")
@@
     ) (layer "B.SilkS") (width 0.007) (fill solid))
   (gr_rect (start 84.8868 95.1738) (end 64.5668 44.323) (layer "Edge.Cuts") (width 0.1) (fill none))
-  (gr_text "   Patrick Pedersen\nTAPR Open Hardware License v1.0" (at 74.69324 61.2902) (layer "B.SilkS")
+  (gr_text "   Patrick Pedersen\nLicensed under CERN-OHL-P v2" (at 74.69324 61.2902) (layer "B.SilkS")
     (effects (font (size 0.7 0.7) (thickness 0.1)) (justify mirror))
   )
